File: hardware/pcb/MStar-WLAN.sch (EAGLE design)
At the start: 41 parts, among them J1 6P6C, J3 ZX62R-B-5P(30), Q1 VP2106, Q2 2N3904

Commit message: pcb
Parts:
- removed 3.3--5V: (no value), jumper:SJ2W
- removed D3: (no value), diode:DIODE-D-5
- removed R8, R9: 10K, rcl:R-US_0207/2V
- C1: value 470u/25 -> 2m/25; device rcl:CPOL-USE3.5-8 -> rcl:CPOL-USE5-10.5
- C2: value 1m/6.3 -> 100u/6.3; device rcl:CPOL-USE5-10.5 -> rcl:CPOL-USE2.5-6
Connections:
- removed net N$16: 3.3--5V.1, D3.A
- removed net N$20: 3.3--5V.2, C2.+, C3.1, OKI-78SR-3.3.OUT
- removed net N$8: ESP32-WROVER-B.SENSOR_VP, R8.1, R9.2
- net GND: no longer R9.1
- net N$17: no longer D3.C
- net VCC: now also C2.+, C3.1, OKI-78SR-3.3.OUT; no longer 3.3--5V.3, R8.2
Other:
- note added: "C1 - United Chemi-Con EGXF250ELL202MJ30S 2000uF/25V"
- note added: "MStar-WLAN 2019.12 mjs"
- note removed: "MStar-WLAN 2019.5 mjs"
Changed lines of the file:
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@@
 <?xml version="1.0" encoding="utf-8"?>
 <!DOCTYPE eagle SYSTEM "eagle.dtd">
-<eagle version="9.3.2">
+<eagle version="9.4.0">
 <drawing>
 <settings>
@@
 <parts>
 <part name="J1" library="con-rj" deviceset="RJ12" device="" value="6P6C"/>
-<part name="C1" library="rcl" deviceset="CPOL-US" device="E3.5-8" value="470u/25"/>
+<part name="C1" library="rcl" deviceset="CPOL-US" device="E5-10.5" value="2m/25"/>
 <part name="R2" library="rcl" deviceset="R-US_" device="0207/2V" value="10K"/>
 <part name="Q1" library="MyLibrary" deviceset="VP2106" device="" value="VP2106"/>
@@
 <part name="R4" library="rcl" deviceset="R-US_" device="0207/2V" value="10K"/>
 <part name="U$1" library="MyLibrary" deviceset="WEMOS-D1-MINI-PRO" device=""/>
-<part name="C2" library="rcl" deviceset="CPOL-US" device="E5-10.5" value="1m/6.3"/>
+<part name="C2" library="rcl" deviceset="CPOL-US" device="E2.5-6" value="100u/6.3"/>
 <part name="MBUS" library="adafruit" library_urn="urn:adsk.eagle:library:420" deviceset="LED" device="3MM" package3d_urn="urn:adsk.eagle:package:6240537/1"/>
 <part name="C10" library="rcl" deviceset="CPOL-US" device="E2.5-5" value="2.2u"/>
@@
 <part name="RESET" library="switch-omron" deviceset="10-XX" device=""/>
 <part name="SUPPLY3" library="supply2" deviceset="GND" device=""/>
-<part name="R9" library="rcl" deviceset="R-US_" device="0207/2V" value="10K"/>
-<part name="R8" library="rcl" deviceset="R-US_" device="0207/2V" value="10K"/>
 <part name="SUPPLY4" library="supply2" deviceset="GND" device=""/>
 <part name="R10" library="rcl" deviceset="R-US_" device="0207/2V" value="27"/>
@@
 <part name="C4" library="rcl" deviceset="C-US" device="025-024X044" value="0.1u"/>
 <part name="C9" library="rcl" deviceset="C-US" device="025-024X044" value="0.1u"/>
-<part name="D3" library="diode" deviceset="DIODE-" device="D-5"/>
 <part name="D4" library="diode" deviceset="DIODE-" device="D-5"/>
-<part name="3.3--5V" library="jumper" deviceset="SJ2W" device=""/>
 <part name="OKI-78SR-3.3" library="v-reg" deviceset="78MXXS" device=""/>
 <part name="DS3231(ZS-042)" library="MyLibrary" deviceset="RTC-DS3231-AT24C32-6" device="" value=""/>
@@
 154-UL6661</text>
 <text x="40.64" y="134.62" size="3.81" layer="91">MStar-WLAN
-2019.5 mjs</text>
+2019.12 mjs</text>
 <text x="177.8" y="149.86" size="3.048" layer="94">WROVER only</text>
+<text x="68.58" y="114.3" size="1.778" layer="94">C1 - United Chemi-Con
+EGXF250ELL202MJ30S
+2000uF/25V</text>
 </plain>
 <instances>
@@
 <attribute name="VALUE" x="178.435" y="116.205" size="1.778" layer="96"/>
 </instance>
-<instance part="R9" gate="G$1" x="180.34" y="81.28" smashed="yes" rot="R90">
-<attribute name="NAME" x="178.8414" y="82.55" size="1.778" layer="95" rot="R90"/>
-<attribute name="VALUE" x="178.562" y="77.47" size="1.778" layer="96" rot="R90"/>
-</instance>
-<instance part="R8" gate="G$1" x="180.34" y="93.98" smashed="yes" rot="R90">
-<attribute name="NAME" x="178.8414" y="87.63" size="1.778" layer="95" rot="R90"/>
-<attribute name="VALUE" x="178.562" y="92.71" size="1.778" layer="96" rot="R90"/>
-</instance>
 <instance part="SUPPLY4" gate="GND" x="261.62" y="91.44" smashed="yes">
 <attribute name="VALUE" x="259.715" y="88.265" size="1.778" layer="96"/>
@@
 <attribute name="VALUE" x="252.984" y="98.171" size="1.778" layer="96" rot="R180"/>
 </instance>
-<instance part="D3" gate="G$1" x="297.18" y="134.62" smashed="yes" rot="R270">
-<attribute name="NAME" x="301.7774" y="132.08" size="1.778" layer="95" rot="R90"/>
-<attribute name="VALUE" x="294.8686" y="132.08" size="1.778" layer="96" rot="R270"/>
-</instance>
 <instance part="D4" gate="G$1" x="297.18" y="96.52" smashed="yes" rot="R90">
 <attribute name="NAME" x="292.5826" y="99.06" size="1.778" layer="95" rot="R270"/>
 <attribute name="VALUE" x="299.4914" y="99.06" size="1.778" layer="96" rot="R90"/>
 </instance>
-<instance part="3.3--5V" gate="G$1" x="111.76" y="134.62" smashed="yes">
-<attribute name="NAME" x="116.459" y="129.54" size="1.778" layer="95" rot="R90"/>
-<attribute name="VALUE" x="114.3" y="132.715" size="1.778" layer="96"/>
-</instance>
 <instance part="OKI-78SR-3.3" gate="A" x="81.28" y="104.14" smashed="yes">
-<attribute name="NAME" x="86.36" y="109.22" size="1.778" layer="95" rot="R180"/>
+<attribute name="NAME" x="88.9" y="109.22" size="1.778" layer="95" rot="R180"/>
 <attribute name="VALUE" x="83.82" y="93.98" size="1.778" layer="96"/>
 </instance>
@@
 <segment>
 <label x="127" y="104.14" size="1.778" layer="95"/>
-<wire x1="111.76" y1="104.14" x2="180.34" y2="104.14" width="0.1524" layer="91"/>
-<wire x1="180.34" y1="104.14" x2="193.04" y2="104.14" width="0.1524" layer="91"/>
+<wire x1="111.76" y1="104.14" x2="193.04" y2="104.14" width="0.1524" layer="91"/>
 <wire x1="193.04" y1="104.14" x2="231.14" y2="104.14" width="0.1524" layer="91"/>
 <pinref part="ESP32-WROVER-B" gate="G$1" pin="VDD3V3"/>
@@
 <junction x="193.04" y="104.14"/>
 <label x="248.92" y="104.14" size="1.778" layer="95"/>
-<pinref part="R8" gate="G$1" pin="2"/>
-<wire x1="180.34" y1="99.06" x2="180.34" y2="104.14" width="0.1524" layer="91"/>
-<junction x="180.34" y="104.14"/>
 <pinref part="C6" gate="G$1" pin="1"/>
 <pinref part="LDL1117S33" gate="G$1" pin="OUT"/>
@@
 <pinref part="C9" gate="G$1" pin="1"/>
 <junction x="254" y="104.14"/>
-<pinref part="3.3--5V" gate="G$1" pin="3"/>
 <wire x1="111.76" y1="104.14" x2="111.76" y2="116.84" width="0.1524" layer="91"/>
 <junction x="111.76" y="104.14"/>
 <pinref part="DS3231(ZS-042)" gate="G$1" pin="VCC.1"/>
-<wire x1="111.76" y1="116.84" x2="111.76" y2="129.54" width="0.1524" layer="91"/>
 <wire x1="127" y1="116.84" x2="111.76" y2="116.84" width="0.1524" layer="91"/>
-<junction x="111.76" y="116.84"/>
 <pinref part="R12" gate="G$1" pin="2"/>
 <wire x1="144.78" y1="43.18" x2="121.92" y2="43.18" width="0.1524" layer="91"/>
 <wire x1="121.92" y1="43.18" x2="121.92" y2="66.04" width="0.1524" layer="91"/>
 <junction x="121.92" y="66.04"/>
+<pinref part="C2" gate="G$1" pin="+"/>
+<wire x1="101.6" y1="104.14" x2="101.6" y2="99.06" width="0.1524" layer="91"/>
+<wire x1="96.52" y1="104.14" x2="101.6" y2="104.14" width="0.1524" layer="91"/>
+<pinref part="C3" gate="G$1" pin="1"/>
+<junction x="96.52" y="104.14"/>
+<wire x1="88.9" y1="104.14" x2="96.52" y2="104.14" width="0.1524" layer="91"/>
+<pinref part="OKI-78SR-3.3" gate="A" pin="OUT"/>
+<wire x1="101.6" y1="104.14" x2="111.76" y2="104.14" width="0.1524" layer="91"/>
+<junction x="101.6" y="104.14"/>
 </segment>
 </net>
@@
 <wire x1="101.6" y1="30.48" x2="83.82" y2="30.48" width="0.1524" layer="91"/>
 <junction x="101.6" y="30.48"/>
-<wire x1="180.34" y1="76.2" x2="180.34" y2="30.48" width="0.1524" layer="91"/>
-<wire x1="180.34" y1="30.48" x2="83.82" y2="30.48" width="0.1524" layer="91"/>
+<wire x1="228.6" y1="30.48" x2="83.82" y2="30.48" width="0.1524" layer="91"/>
 <junction x="83.82" y="30.48"/>
-<junction x="180.34" y="30.48"/>
-<wire x1="180.34" y1="30.48" x2="228.6" y2="30.48" width="0.1524" layer="91"/>
 <wire x1="228.6" y1="30.48" x2="228.6" y2="38.1" width="0.1524" layer="91"/>
 <pinref part="ESP32-WROVER-B" gate="G$1" pin="GND"/>
@@
 <pinref part="SUPPLY1" gate="GND" pin="GND"/>
 <junction x="58.42" y="30.48"/>
-<pinref part="R9" gate="G$1" pin="1"/>
 <pinref part="C2" gate="G$1" pin="-"/>
 <wire x1="101.6" y1="86.36" x2="101.6" y2="91.44" width="0.1524" layer="91"/>
@@
 </segment>
 </net>
-<net name="N$8" class="0">
-<segment>
-<pinref part="R8" gate="G$1" pin="1"/>
-<pinref part="R9" gate="G$1" pin="2"/>
-<wire x1="180.34" y1="88.9" x2="180.34" y2="86.36" width="0.1524" layer="91"/>
-<pinref part="ESP32-WROVER-B" gate="G$1" pin="SENSOR_VP"/>
-<wire x1="195.58" y1="86.36" x2="180.34" y2="86.36" width="0.1524" layer="91"/>
-<junction x="180.34" y="86.36"/>
-</segment>
-</net>
 <net name="N$9" class="0">
 <segment>
@@
 </segment>
 </net>
-<net name="N$16" class="1">
-<segment>
-<wire x1="297.18" y1="147.32" x2="297.18" y2="137.16" width="0.1524" layer="91"/>
-<pinref part="D3" gate="G$1" pin="A"/>
-<pinref part="3.3--5V" gate="G$1" pin="1"/>
-<wire x1="297.18" y1="147.32" x2="111.76" y2="147.32" width="0.1524" layer="91"/>
-<wire x1="111.76" y1="147.32" x2="111.76" y2="139.7" width="0.1524" layer="91"/>
-</segment>
-</net>
 <net name="N$17" class="1">
 <segment>
@@
 <pinref part="D4" gate="G$1" pin="C"/>
 <wire x1="297.18" y1="99.06" x2="297.18" y2="114.3" width="0.1524" layer="91"/>
-<pinref part="D3" gate="G$1" pin="C"/>
-<wire x1="297.18" y1="132.08" x2="297.18" y2="114.3" width="0.1524" layer="91"/>
-<junction x="297.18" y="114.3"/>
-</segment>
-</net>
-<net name="N$20" class="1">
-<segment>
-<pinref part="C2" gate="G$1" pin="+"/>
-<wire x1="101.6" y1="104.14" x2="101.6" y2="99.06" width="0.1524" layer="91"/>
-<wire x1="96.52" y1="104.14" x2="101.6" y2="104.14" width="0.1524" layer="91"/>
-<pinref part="C3" gate="G$1" pin="1"/>
-<junction x="96.52" y="104.14"/>
-<wire x1="88.9" y1="104.14" x2="96.52" y2="104.14" width="0.1524" layer="91"/>
-<wire x1="101.6" y1="104.14" x2="101.6" y2="134.62" width="0.1524" layer="91"/>
-<junction x="101.6" y="104.14"/>
-<pinref part="3.3--5V" gate="G$1" pin="2"/>
-<wire x1="101.6" y1="134.62" x2="106.68" y2="134.62" width="0.1524" layer="91"/>
-<pinref part="OKI-78SR-3.3" gate="A" pin="OUT"/>
-</segment>
-</net>
+</segment>
+</net>

Commit message: ESP32 work
Parts:
- added C11: 10u, rcl:C-USC1206
- added SD: (no value), con-lsta:FE06-1
Connections:
- new net N$16: ESP32-WROVER-B.IO5, SD.2
- new net N$20: ESP32-WROVER-B.IO18, SD.4
- new net N$22: ESP32-WROVER-B.IO23, SD.3
- new net N$8: ESP32-WROVER-B.IO19, SD.5
- net GND: now also C11.2, SD.6
- net RX_ENA: now also ESP32-WROVER-B.IO25; no longer ESP32-WROVER-B.IO23
- net VCC: now also C11.1, SD.1
Other:
- note added: "3v3"
- note added: "CLK"
- note added: "CS"
- note added: "GND"
- note added: "MISO"
- note added: "MOSI"
Changed lines of the file:
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@@
 <part name="SUPPLY6" library="supply2" deviceset="GND" device=""/>
 <part name="SUPPLY7" library="supply2" deviceset="GND" device=""/>
+<part name="SD" library="con-lsta" library_urn="urn:adsk.eagle:library:161" deviceset="FE06-1" device="" package3d_urn="urn:adsk.eagle:package:8191/1"/>
+<part name="C11" library="rcl" deviceset="C-US" device="C1206" value="10u"/>
 </parts>
 <sheets>
@@
 EGXF250ELL202MJ30S
 2000uF/25V</text>
+<text x="186.436" y="6.35" size="1.778" layer="91" rot="R90">3v3</text>
+<text x="189.23" y="6.858" size="1.778" layer="91" rot="R90">CS</text>
+<text x="191.77" y="4.318" size="1.778" layer="91" rot="R90">MOSI</text>
+<text x="194.31" y="5.588" size="1.778" layer="91" rot="R90">CLK</text>
+<text x="196.85" y="4.318" size="1.778" layer="91" rot="R90">MISO</text>
+<text x="199.39" y="5.08" size="1.778" layer="91" rot="R90">GND</text>
 </plain>
 <instances>
@@
 <instance part="R11" gate="G$1" x="304.8" y="55.88" smashed="yes" rot="R180">
 <attribute name="NAME" x="306.324" y="62.0014" size="1.778" layer="95" rot="R180"/>
-<attribute name="VALUE" x="306.832" y="51.816" size="1.778" layer="96" rot="R180"/>
+<attribute name="VALUE" x="306.832" y="64.516" size="1.778" layer="96" rot="R180"/>
 </instance>
 <instance part="C3" gate="G$1" x="96.52" y="101.6" smashed="yes">
@@
 </instance>
 <instance part="SUPPLY7" gate="GND" x="165.1" y="58.42" smashed="yes">
-<attribute name="VALUE" x="163.195" y="55.245" size="1.778" layer="96"/>
+<attribute name="VALUE" x="164.465" y="61.595" size="1.778" layer="96" rot="R180"/>
+</instance>
+<instance part="SD" gate="G$1" x="190.5" y="12.7" smashed="yes" rot="MR90">
+<attribute name="VALUE" x="180.34" y="11.43" size="1.778" layer="96" rot="MR90"/>
+<attribute name="NAME" x="201.422" y="11.43" size="1.778" layer="95" rot="MR90"/>
+</instance>
+<instance part="C11" gate="G$1" x="180.34" y="25.4" smashed="yes" rot="R180">
+<attribute name="NAME" x="179.324" y="24.765" size="1.778" layer="95" rot="R180"/>
+<attribute name="VALUE" x="179.324" y="29.591" size="1.778" layer="96" rot="R180"/>
 </instance>
 </instances>
@@
 <wire x1="124.46" y1="68.58" x2="124.46" y2="53.34" width="0.1524" layer="91"/>
 <junction x="124.46" y="53.34"/>
-<wire x1="124.46" y1="53.34" x2="190.5" y2="53.34" width="0.1524" layer="91"/>
+<wire x1="124.46" y1="53.34" x2="180.34" y2="53.34" width="0.1524" layer="91"/>
 <pinref part="ESP32-WROVER-B" gate="G$1" pin="IO4"/>
-<wire x1="190.5" y1="53.34" x2="190.5" y2="73.66" width="0.1524" layer="91"/>
-<wire x1="190.5" y1="73.66" x2="195.58" y2="73.66" width="0.1524" layer="91"/>
-<label x="127" y="53.34" size="1.778" layer="95"/>
+<wire x1="180.34" y1="53.34" x2="180.34" y2="73.66" width="0.1524" layer="91"/>
+<wire x1="180.34" y1="73.66" x2="195.58" y2="73.66" width="0.1524" layer="91"/>
+<label x="167.64" y="53.34" size="1.778" layer="95"/>
 </segment>
 </net>
@@
 <wire x1="127" y1="116.84" x2="111.76" y2="116.84" width="0.1524" layer="91"/>
 <pinref part="R12" gate="G$1" pin="2"/>
-<wire x1="144.78" y1="43.18" x2="121.92" y2="43.18" width="0.1524" layer="91"/>
+<wire x1="144.78" y1="43.18" x2="139.7" y2="43.18" width="0.1524" layer="91"/>
+<wire x1="139.7" y1="43.18" x2="121.92" y2="43.18" width="0.1524" layer="91"/>
 <wire x1="121.92" y1="43.18" x2="121.92" y2="66.04" width="0.1524" layer="91"/>
 <junction x="121.92" y="66.04"/>
@@
 <wire x1="101.6" y1="104.14" x2="111.76" y2="104.14" width="0.1524" layer="91"/>
 <junction x="101.6" y="104.14"/>
+<wire x1="139.7" y1="43.18" x2="139.7" y2="22.86" width="0.1524" layer="91"/>
+<junction x="139.7" y="43.18"/>
+<wire x1="139.7" y1="22.86" x2="180.34" y2="22.86" width="0.1524" layer="91"/>
+<pinref part="SD" gate="G$1" pin="1"/>
+<wire x1="180.34" y1="22.86" x2="185.42" y2="22.86" width="0.1524" layer="91"/>
+<wire x1="185.42" y1="22.86" x2="185.42" y2="20.32" width="0.1524" layer="91"/>
+<pinref part="C11" gate="G$1" pin="1"/>
+<junction x="180.34" y="22.86"/>
 </segment>
 </net>
@@
 <junction x="116.84" y="45.72"/>
 <wire x1="116.84" y1="33.02" x2="231.14" y2="33.02" width="0.1524" layer="91"/>
-<label x="127" y="33.02" size="1.778" layer="95"/>
+<label x="165.1" y="33.02" size="1.778" layer="95"/>
 <wire x1="231.14" y1="33.02" x2="231.14" y2="48.26" width="0.1524" layer="91"/>
 <pinref part="ESP32-WROVER-B" gate="G$1" pin="IO27"/>
@@
 <wire x1="101.6" y1="30.48" x2="83.82" y2="30.48" width="0.1524" layer="91"/>
 <junction x="101.6" y="30.48"/>
-<wire x1="228.6" y1="30.48" x2="83.82" y2="30.48" width="0.1524" layer="91"/>
+<wire x1="228.6" y1="30.48" x2="198.12" y2="30.48" width="0.1524" layer="91"/>
 <junction x="83.82" y="30.48"/>
+<wire x1="198.12" y1="30.48" x2="180.34" y2="30.48" width="0.1524" layer="91"/>
+<wire x1="180.34" y1="30.48" x2="83.82" y2="30.48" width="0.1524" layer="91"/>
 <wire x1="228.6" y1="30.48" x2="228.6" y2="38.1" width="0.1524" layer="91"/>
 <pinref part="ESP32-WROVER-B" gate="G$1" pin="GND"/>
@@
 <wire x1="81.28" y1="96.52" x2="81.28" y2="93.98" width="0.1524" layer="91"/>
 <junction x="81.28" y="93.98"/>
+<pinref part="SD" gate="G$1" pin="6"/>
+<wire x1="198.12" y1="20.32" x2="198.12" y2="30.48" width="0.1524" layer="91"/>
+<junction x="198.12" y="30.48"/>
+<pinref part="C11" gate="G$1" pin="2"/>
+<junction x="180.34" y="30.48"/>
 </segment>
 <segment>
@@
 <wire x1="114.3" y1="73.66" x2="101.6" y2="73.66" width="0.1524" layer="91"/>
 <wire x1="101.6" y1="73.66" x2="101.6" y2="71.12" width="0.1524" layer="91"/>
-<wire x1="114.3" y1="73.66" x2="114.3" y2="48.26" width="0.1524" layer="91"/>
+<wire x1="114.3" y1="73.66" x2="114.3" y2="50.8" width="0.1524" layer="91"/>
 <junction x="114.3" y="73.66"/>
-<wire x1="195.58" y1="48.26" x2="114.3" y2="48.26" width="0.1524" layer="91"/>
-<label x="127" y="48.26" size="1.778" layer="95"/>
-<pinref part="ESP32-WROVER-B" gate="G$1" pin="IO23"/>
+<label x="162.56" y="50.8" size="1.778" layer="95"/>
+<wire x1="114.3" y1="50.8" x2="180.34" y2="50.8" width="0.1524" layer="91"/>
+<pinref part="ESP32-WROVER-B" gate="G$1" pin="IO25"/>
+<wire x1="195.58" y1="45.72" x2="180.34" y2="45.72" width="0.1524" layer="91"/>
+<wire x1="180.34" y1="45.72" x2="180.34" y2="50.8" width="0.1524" layer="91"/>
 </segment>
 </net>
@@
 <net name="N$19" class="0">
 <segment>
-<wire x1="187.96" y1="71.12" x2="172.72" y2="71.12" width="0.1524" layer="91"/>
+<wire x1="177.8" y1="71.12" x2="172.72" y2="71.12" width="0.1524" layer="91"/>
 <pinref part="WLAN" gate="G$1" pin="C"/>
 <wire x1="172.72" y1="71.12" x2="172.72" y2="43.18" width="0.1524" layer="91"/>
 <wire x1="172.72" y1="43.18" x2="165.1" y2="43.18" width="0.1524" layer="91"/>
 <pinref part="ESP32-WROVER-B" gate="G$1" pin="IO2"/>
-<wire x1="195.58" y1="76.2" x2="187.96" y2="76.2" width="0.1524" layer="91"/>
-<wire x1="187.96" y1="76.2" x2="187.96" y2="71.12" width="0.1524" layer="91"/>
+<wire x1="195.58" y1="76.2" x2="177.8" y2="76.2" width="0.1524" layer="91"/>
+<wire x1="177.8" y1="76.2" x2="177.8" y2="71.12" width="0.1524" layer="91"/>
 <pinref part="U$1" gate="G$1" pin="D4"/>
 <wire x1="162.56" y1="71.12" x2="172.72" y2="71.12" width="0.1524" layer="91"/>
@@
 <pinref part="ESP32-WROVER-B" gate="G$1" pin="IO14"/>
 <wire x1="119.38" y1="76.2" x2="114.3" y2="76.2" width="0.1524" layer="91"/>
-<wire x1="195.58" y1="63.5" x2="193.04" y2="63.5" width="0.1524" layer="91"/>
-<wire x1="193.04" y1="63.5" x2="193.04" y2="38.1" width="0.1524" layer="91"/>
-<wire x1="193.04" y1="38.1" x2="119.38" y2="38.1" width="0.1524" layer="91"/>
+<wire x1="195.58" y1="63.5" x2="182.88" y2="63.5" width="0.1524" layer="91"/>
+<wire x1="182.88" y1="63.5" x2="182.88" y2="38.1" width="0.1524" layer="91"/>
+<wire x1="182.88" y1="38.1" x2="119.38" y2="38.1" width="0.1524" layer="91"/>
 <wire x1="119.38" y1="38.1" x2="119.38" y2="76.2" width="0.1524" layer="91"/>
 <junction x="119.38" y="76.2"/>
@@
 <wire x1="114.3" y1="124.46" x2="127" y2="124.46" width="0.1524" layer="91"/>
 <label x="114.3" y="76.2" size="1.778" layer="95"/>
-<label x="127" y="38.1" size="1.778" layer="95"/>
+<label x="165.1" y="38.1" size="1.778" layer="95"/>
 </segment>
 </net>
@@
 </segment>
 </net>
+<net name="N$8" class="0">
+<segment>
+<pinref part="SD" gate="G$1" pin="5"/>
+<pinref part="ESP32-WROVER-B" gate="G$1" pin="IO19"/>
+<wire x1="195.58" y1="20.32" x2="195.58" y2="27.94" width="0.1524" layer="91"/>
+<wire x1="195.58" y1="27.94" x2="187.96" y2="27.94" width="0.1524" layer="91"/>
+<wire x1="187.96" y1="27.94" x2="187.96" y2="55.88" width="0.1524" layer="91"/>
+<wire x1="187.96" y1="55.88" x2="195.58" y2="55.88" width="0.1524" layer="91"/>
+</segment>
+</net>
+<net name="N$16" class="0">
+<segment>
+<pinref part="ESP32-WROVER-B" gate="G$1" pin="IO5"/>
+<wire x1="195.58" y1="71.12" x2="185.42" y2="71.12" width="0.1524" layer="91"/>
+<wire x1="185.42" y1="71.12" x2="185.42" y2="25.4" width="0.1524" layer="91"/>
+<wire x1="185.42" y1="25.4" x2="187.96" y2="25.4" width="0.1524" layer="91"/>
+<pinref part="SD" gate="G$1" pin="2"/>
+<wire x1="187.96" y1="25.4" x2="187.96" y2="20.32" width="0.1524" layer="91"/>
+</segment>
+</net>
+<net name="N$20" class="0">
+<segment>
+<pinref part="ESP32-WROVER-B" gate="G$1" pin="IO18"/>
+<wire x1="195.58" y1="58.42" x2="193.04" y2="58.42" width="0.1524" layer="91"/>
+<wire x1="193.04" y1="58.42" x2="193.04" y2="20.32" width="0.1524" layer="91"/>
+<pinref part="SD" gate="G$1" pin="4"/>
+</segment>
+</net>
+<net name="N$22" class="0">
+<segment>
+<pinref part="ESP32-WROVER-B" gate="G$1" pin="IO23"/>
+<wire x1="195.58" y1="48.26" x2="190.5" y2="48.26" width="0.1524" layer="91"/>
+<wire x1="190.5" y1="48.26" x2="190.5" y2="20.32" width="0.1524" layer="91"/>
+<pinref part="SD" gate="G$1" pin="3"/>
+</segment>
+</net>
